File: pcb/driver.sch (KiCad schematic (older format))
At the start: 22 parts, among them Q1 Q_NMOS_GDS, U1 AL8853

Commit message: added firmware and updated driver pcnb
Parts:
- removed C1, C2: 100n, Capacitor_SMD:C_0603_1608Metric_Pad1.05x0.95mm_HandSolder, symbol Device:C
- removed C3: 4.7u, Capacitor_THT:C_Radial_D10.0mm_H16.0mm_P5.00mm, symbol Device:C
- removed C4: 470u, Capacitor_SMD:C_Elec_10x10.2, symbol Device:C
- removed D1: MBRB40250TG, Package_TO_SOT_SMD:TO-263-3_TabPin4, symbol Diode:MBRB40250TG
- removed GND1, Vin1: Conn_01x01_Female, Connector_Wire:SolderWirePad_1x01_SMD_5x10mm, symbol Connector:Conn_01x01_Female
- removed GND2, JLED+1, JLED-1, PWMin1, Vin2: Conn_01x01_Female, Connector_Wire:SolderWirePad_1x01_SMD_1x2mm, symbol Connector:Conn_01x01_Female
- removed L1: Lx, Inductor_SMD:L_17x17_H7, symbol Device:L
- removed L2: Ls, Inductor_SMD:L_12x12mm_H8mm, symbol Device:L
- removed Q1: Q_NMOS_GDS, Package_TO_SOT_SMD:SOT-223-3_TabPin2, symbol Device:Q_NMOS_GDS
- removed R4: 170k, Resistor_SMD:R_0603_1608Metric_Pad1.05x0.95mm_HandSolder, symbol Device:R
- removed R5, RPWM1: 10k, Resistor_SMD:R_0603_1608Metric_Pad1.05x0.95mm_HandSolder, symbol Device:R
- removed Rfb1: 1.33, Resistor_SMD:R_0805_2012Metric_Pad1.15x1.40mm_HandSolder, symbol Device:R
- removed Rocp1, Rocp2: Rocp, Resistor_SMD:R_2512_6332Metric_Pad1.52x3.35mm_HandSolder, symbol Device:R
- removed U1: AL8853, Package_SO:SO-8_5.3x6.2mm_P1.27mm, symbol Driver_LED:AL8853
