File: pcb/lamp10.sch (KiCad schematic (older format))
At the start: 12 parts, among them J1 Conn_01x01_Female, J2 Conn_01x01_Female

Commit message: added firmware and updated driver pcnb
Parts:
- removed D1, D10, D2, D3, D4, D5, D6, D7, D8, D9: LED, LED_SMD:LED_PLCC_2835_Handsoldering, symbol Device:LED
- removed J1, J2: Conn_01x01_Female, Connector_Wire:SolderWirePad_1x01_SMD_1x2mm, symbol Connector:Conn_01x01_Female
Changed lines of the file:
@@
 $Descr A4 11693 8268
 encoding utf-8
-Sheet 1 1
+Sheet 1 6
 Title ""
 Date ""
@@
 Comment4 ""
 $EndDescr
-$Comp
-L Connector:Conn_01x01_Female J2
-U 1 1 5FEE7107
-P 4900 3250
-F 0 "J2" H 4928 3276 50  0000 L CNN
-F 1 "Conn_01x01_Female" H 4928 3185 50  0000 L CNN
-F 2 "Connector_Wire:SolderWirePad_1x01_SMD_1x2mm" H 4900 3250 50  0001 C CNN
-F 3 "~" H 4900 3250 50  0001 C CNN
-	1    4900 3250
-	1    0    0    -1
-$EndComp
-$Comp
-L Device:LED D1
-U 1 1 5FEE7761
-P 4700 3400
-F 0 "D1" V 4739 3282 50  0000 R CNN
-F 1 "LED" V 4648 3282 50  0000 R CNN
-F 2 "LED_SMD:LED_PLCC_2835_Handsoldering" H 4700 3400 50  0001 C CNN
-F 3 "~" H 4700 3400 50  0001 C CNN
-	1    4700 3400
-	0    -1   -1   0
-$EndComp
-Text GLabel 4700 3250 1    50   Input ~ 0
-LED+
-$Comp
-L Device:LED D2
-U 1 1 5FEE8F51
-P 4700 3700
-F 0 "D2" V 4739 3582 50  0000 R CNN
-F 1 "LED" V 4648 3582 50  0000 R CNN
-F 2 "LED_SMD:LED_PLCC_2835_Handsoldering" H 4700 3700 50  0001 C CNN
-F 3 "~" H 4700 3700 50  0001 C CNN
-	1    4700 3700
-	0    -1   -1   0
-$EndComp
-$Comp
-L Device:LED D3
-U 1 1 5FEE985E
-P 4700 4000
-F 0 "D3" V 4739 3882 50  0000 R CNN
-F 1 "LED" V 4648 3882 50  0000 R CNN
-F 2 "LED_SMD:LED_PLCC_2835_Handsoldering" H 4700 4000 50  0001 C CNN
-F 3 "~" H 4700 4000 50  0001 C CNN
-	1    4700 4000
-	0    -1   -1   0
-$EndComp
-$Comp
-L Device:LED D4
-U 1 1 5FEE9C35
-P 4700 4300
-F 0 "D4" V 4739 4182 50  0000 R CNN
-F 1 "LED" V 4648 4182 50  0000 R CNN
-F 2 "LED_SMD:LED_PLCC_2835_Handsoldering" H 4700 4300 50  0001 C CNN
-F 3 "~" H 4700 4300 50  0001 C CNN
-	1    4700 4300
-	0    -1   -1   0
-$EndComp
-$Comp
-L Device:LED D5
-U 1 1 5FEEA3AC
-P 4700 4600
-F 0 "D5" V 4739 4482 50  0000 R CNN
-F 1 "LED" V 4648 4482 50  0000 R CNN
-F 2 "LED_SMD:LED_PLCC_2835_Handsoldering" H 4700 4600 50  0001 C CNN
-F 3 "~" H 4700 4600 50  0001 C CNN
-	1    4700 4600
-	0    -1   -1   0
-$EndComp
-$Comp
-L Device:LED D6
-U 1 1 5FEF4A45
-P 4700 4900
-F 0 "D6" V 4739 4782 50  0000 R CNN
-F 1 "LED" V 4648 4782 50  0000 R CNN
-F 2 "LED_SMD:LED_PLCC_2835_Handsoldering" H 4700 4900 50  0001 C CNN
-F 3 "~" H 4700 4900 50  0001 C CNN
-	1    4700 4900
-	0    -1   -1   0
-$EndComp
-$Comp
-L Device:LED D7
-U 1 1 5FEF4A4B
-P 4700 5200
-F 0 "D7" V 4739 5082 50  0000 R CNN
-F 1 "LED" V 4648 5082 50  0000 R CNN
-F 2 "LED_SMD:LED_PLCC_2835_Handsoldering" H 4700 5200 50  0001 C CNN
-F 3 "~" H 4700 5200 50  0001 C CNN
-	1    4700 5200
-	0    -1   -1   0
-$EndComp
-$Comp
-L Device:LED D8
-U 1 1 5FEF4A51
-P 4700 5500
-F 0 "D8" V 4739 5382 50  0000 R CNN
-F 1 "LED" V 4648 5382 50  0000 R CNN
-F 2 "LED_SMD:LED_PLCC_2835_Handsoldering" H 4700 5500 50  0001 C CNN
-F 3 "~" H 4700 5500 50  0001 C CNN
-	1    4700 5500
-	0    -1   -1   0
-$EndComp
-$Comp
-L Device:LED D9
-U 1 1 5FEF4A57
-P 4700 5800
-F 0 "D9" V 4739 5682 50  0000 R CNN
-F 1 "LED" V 4648 5682 50  0000 R CNN
-F 2 "LED_SMD:LED_PLCC_2835_Handsoldering" H 4700 5800 50  0001 C CNN
-F 3 "~" H 4700 5800 50  0001 C CNN
-	1    4700 5800
-	0    -1   -1   0
-$EndComp
-$Comp
-L Device:LED D10
-U 1 1 5FEF4A5D
-P 4700 6100
-F 0 "D10" V 4739 5982 50  0000 R CNN
-F 1 "LED" V 4648 5982 50  0000 R CNN
-F 2 "LED_SMD:LED_PLCC_2835_Handsoldering" H 4700 6100 50  0001 C CNN
-F 3 "~" H 4700 6100 50  0001 C CNN
-	1    4700 6100
-	0    -1   -1   0
-$EndComp
-$Comp
-L Connector:Conn_01x01_Female J1
-U 1 1 5FEE72EA
-P 4700 6450
-F 0 "J1" V 4546 6498 50  0000 L CNN
-F 1 "Conn_01x01_Female" V 4637 6498 50  0000 L CNN
-F 2 "Connector_Wire:SolderWirePad_1x01_SMD_1x2mm" H 4700 6450 50  0001 C CNN
-F 3 "~" H 4700 6450 50  0001 C CNN
-	1    4700 6450
-	0    1    1    0
-$EndComp
-Text GLabel 4700 6250 0    50   Input ~ 0
-LED-
 $EndSCHEMATC
