File: pcb/lampe.sch (KiCad schematic (older format))
At the start: 10 parts

Commit message: added firmware and updated driver pcnb
Changed lines of the file:
@@
 $Descr A4 11693 8268
 encoding utf-8
-Sheet 1 5
+Sheet 1 6
 Title ""
 Date ""
@@
 F1 "lamp60.sch" 50
 $EndSheet
+$Sheet
+S 5800 -5650 3100 1250
+U 5FEF9579
+F0 "driver-v2" 50
+F1 "driver-v2/driver-v2.sch" 50
+$EndSheet
 $EndSCHEMATC
